Commit message: Added hex_ft_sensor and world

File: urdf/ur.ros2_control.xacro (robot description, xacro)
@@ -28,5 +28,5 @@
         </xacro:if>
         <xacro:if value="${sim_ignition}">
-          <plugin>ign_ros2_control/IgnitionSystem</plugin>
+          <plugin>gz_ros2_control/GazeboSimSystem</plugin>
         </xacro:if>
         <xacro:if value="${use_fake_hardware}">

File: urdf/ur_macro.xacro (robot description, xacro)
@@ -48,4 +48,5 @@
     tf_prefix
     parent
+    mount_yaw
     *origin
     joint_limits_parameters_file
@@ -316,5 +317,5 @@
     <!-- base_joint fixes base_link to the environment -->
     <joint name="${tf_prefix}base_joint" type="fixed">
-      <xacro:insert_block name="origin" />
+      <origin xyz="0 0 0" rpy="0 0 ${mount_yaw}" />
       <parent link="${parent}" />
       <child link="${tf_prefix}base_link" />

File: urdf/ur_on_rail.urdf.xacro (robot description, xacro)
@@ -11,4 +11,5 @@
   <xacro:property name="stand_depth" value="0.5" />
   <xacro:property name="stand_height" value="0.8" />
+  <xacro:property name="slider_height" value="0.05" />
   <xacro:arg name="name" default="ur" />
   <!-- import main macro -->
@@ -67,28 +68,26 @@
   <!-- create link fixed to the "world" -->
   <link name="world" />
-  <xacro:if value="${is_sim_gazebo or is_sim_ignition}">
-    <link name="ground_plane">
-      <visual>
-        <origin rpy="0 0 0" xyz="0 0 0" />
-        <geometry>
-          <box size="100 100 0.001" />
-        </geometry>
-        <material name="ground_white">
-          <color rgba="1 1 1 0.5" />
-        </material>
-      </visual>
-      <collision>
-        <origin rpy="0 0 0" xyz="0 0 0" />
-        <geometry>
-          <box size="100 100 0.001" />
-        </geometry>
-      </collision>
-    </link>
-    <joint name="ground_plane_joint" type="fixed">
-      <origin xyz="0 0 -0.01" rpy="0 0 0" />
-      <parent link="world" />
-      <child link="ground_plane" />
-    </joint>
-  </xacro:if>
+  <link name="work_cell">
+    <visual>
+      <origin rpy="0 0 1.5707" xyz="0 0 -0.1" />
+      <geometry>
+        <mesh filename="file://$(find ur_rail_description)/meshes/workspace/work_cell.stl" scale="0.001 0.001 0.001"/>
+      </geometry>
+      <material name="ground_black">
+        <color rgba="0.1 0.1 0.1 1.0" />
+      </material>
+    </visual>
+    <collision>
+      <origin rpy="0 0 1.5707" xyz="0 0 -0.1" />
+      <geometry>
+        <mesh filename="file://$(find ur_rail_description)/meshes/workspace/work_cell.stl" scale="0.001 0.001 0.001"/>
+      </geometry>
+    </collision>
+  </link>
+  <joint name="work_cell_joint" type="fixed">
+    <origin xyz="0 0 0" rpy="0 0 0" />
+    <parent link="world" />
+    <child link="work_cell" />
+  </joint>
   <!-- arm -->
   <xacro:ur_robot
@@ -96,4 +95,5 @@
     tf_prefix="$(arg tf_prefix)"
     parent="slider_base"
+    mount_yaw="0.7854"
     joint_limits_parameters_file="$(arg joint_limit_params)"
     kinematics_parameters_file="$(arg kinematics_params)"
@@ -127,121 +127,140 @@
     reverse_port="$(arg reverse_port)"
     script_sender_port="$(arg script_sender_port)"
-    trajectory_port="$(arg trajectory_port)"
-  >
-    <origin xyz="0 0 0" rpy="0 0 0" />          <!-- position robot in the world -->
+    trajectory_port="$(arg trajectory_port)">
+    <origin xyz="0 0 0" rpy="0 0 0" />
   </xacro:ur_robot>
-  <link name="stand_base">
-    <visual>
-      <origin xyz="0 0 ${stand_height/2}" rpy="0 0 0" />
-      <geometry>
-        <box size="${stand_width} ${stand_depth} ${stand_height}" />
-      </geometry>
-      <material name="Gray">
-        <color rgba="0.7 0.7 0.7 1.0" />
-      </material>
-    </visual>
-    <collision>
-      <origin xyz="0 0 ${stand_height/2}" rpy="0 0 0" />
-      <geometry>
-        <box size="${stand_width} ${stand_depth} ${stand_height}" />
-      </geometry>
-    </collision>
-    <inertial>
-      <mass value="10.0" />
-      <inertia ixx="1.0" ixy="0.0" ixz="0.0" iyy="1.0" iyz="0.0" izz="1.0" />
-    </inertial>
-  </link>
-  <!-- Stand legs -->
-  <link name="stand_leg_1">
-    <visual>
-      <origin xyz="0 0 0" rpy="0 0 0" />
-      <geometry>
-        <cylinder radius="0.05" length="${stand_height*0.1}" />
+  <link name="hex_qc_ft_sensor">
+    <visual>
+      <origin xyz="-0.058 -0.02 -0.03" rpy="1.5707 0 3.1414" />
+      <geometry>
+        <mesh filename="file://$(find ur_rail_description)/meshes/onrobot_hex_qc_rg2/visual/HEX_E_H_QC_v3.dae" scale="0.001 0.001 0.001"/>
+      </geometry>
+      <material name="White">
+        <color rgba="0.79 0.79 0.79 1.0" />
+      </material>
+    </visual>
+    <collision>
+      <origin xyz="-0.058 -0.02 -0.03" rpy="1.5707 0 3.1414" />
+      <geometry>
+        <mesh filename="file://$(find ur_rail_description)/meshes/onrobot_hex_qc_rg2/collision/HEX_E_H_QC_v3.stl" scale="0.001 0.0015 0.001"/>
+      </geometry>
+    </collision>
+    <inertial>
+      <mass value="10.0" />
+      <inertia ixx="1.0" ixy="0.0" ixz="0.0" iyy="1.0" iyz="0.0" izz="1.0" />
+    </inertial>
+  </link>
+  <joint name="ft_tool_joint" type="fixed">
+    <parent link="tool0" />
+    <child link="hex_qc_ft_sensor" />
+    <origin xyz="0 0 0" rpy="0 0 0" />
+  </joint>
+  <link name="plc_linear_rail">
+    <visual>
+      <origin xyz="0 0 0.884" rpy="0 0 0" />
+      <geometry>
+        <mesh filename="file://$(find ur_rail_description)/meshes/workspace/plc_linear_rail.stl" scale="0.001 0.001 0.001"/>
+      </geometry>
+      <material name="White">
+        <color rgba="0.79 0.79 0.79 1.0" />
+      </material>
+    </visual>
+    <collision>
+      <origin xyz="0 0 0.884" rpy="0 0 0" />
+      <geometry>
+        <mesh filename="file://$(find ur_rail_description)/meshes/workspace/plc_linear_rail.stl" scale="0.001 0.001 0.001"/>
+      </geometry>
+    </collision>
+    <inertial>
+      <mass value="10.0" />
+      <inertia ixx="1.0" ixy="0.0" ixz="0.0" iyy="1.0" iyz="0.0" izz="1.0" />
+    </inertial>
+  </link>
+  <!-- Connect plc to world -->
+  <joint name="gnd_plc_joint" type="fixed">
+    <parent link="work_cell" />
+    <child link="plc_linear_rail" />
+    <origin xyz="0.5 -1.03 0" rpy="0 0 1.5707" />
+  </joint>
+  <link name="table1">
+    <visual>
+      <origin xyz="0 0 0" rpy="0 0 0" />
+      <geometry>
+        <mesh filename="file://$(find ur_rail_description)/meshes/workspace/table.stl" scale="0.001 0.001 0.001"/>
+      </geometry>
+      <material name="Aluminium">
+        <color rgba="0.78 0.78 0.78 1.0" />
+      </material>
+    </visual>
+    <collision>
+      <origin xyz="0 0 0" rpy="0 0 0" />
+      <geometry>
+        <mesh filename="file://$(find ur_rail_description)/meshes/workspace/table.stl" scale="0.001 0.001 0.001"/>
+      </geometry>
+    </collision>
+    <inertial>
+      <mass value="10.0" />
+      <inertia ixx="1.0" ixy="0.0" ixz="0.0" iyy="1.0" iyz="0.0" izz="1.0" />
+    </inertial>
+  </link>
+  <link name="table2">
+    <visual>
+      <origin xyz="0 0 0" rpy="0 0 0" />
+      <geometry>
+        <mesh filename="file://$(find ur_rail_description)/meshes/workspace/table.stl" scale="0.001 0.001 0.001"/>
+      </geometry>
+      <material name="Aluminium">
+        <color rgba="0.78 0.78 0.78 1.0" />
+      </material>
+    </visual>
+    <collision>
+      <origin xyz="0 0 0" rpy="0 0 0" />
+      <geometry>
+        <mesh filename="file://$(find ur_rail_description)/meshes/workspace/table.stl" scale="0.001 0.001 0.001"/>
+      </geometry>
+    </collision>
+    <inertial>
+      <mass value="10.0" />
+      <inertia ixx="1.0" ixy="0.0" ixz="0.0" iyy="1.0" iyz="0.0" izz="1.0" />
+    </inertial>
+  </link>
+  <!-- Connect table1 to world -->
+  <joint name="gnd_table1_joint" type="fixed">
+    <parent link="work_cell" />
+    <child link="table1" />
+    <origin xyz="0.34 0.3 0.74" rpy="0 0 0" />
+  </joint>
+  <!-- Connect table2 to world -->
+  <joint name="gnd_table2_joint" type="fixed">
+    <parent link="work_cell" />
+    <child link="table2" />
+    <origin xyz="-0.34 0.3 0.74" rpy="0 0 0" />
+  </joint>
+  <link name="linear_rail">
+    <visual>
+      <origin xyz="0 0 0" rpy="0 0 0" />
+      <geometry>
+        <mesh filename="file://$(find ur_rail_description)/meshes/workspace/linear_rail.stl" scale="0.001 0.001 0.001"/>
       </geometry>
       <material name="DarkGray">
-        <color rgba="0.3 0.3 0.3 1.0" />
-      </material>
-    </visual>
-  </link>
-  <joint name="stand_to_leg_1" type="fixed">
-    <parent link="stand_base" />
-    <child link="stand_leg_1" />
-    <origin xyz="${-stand_width/2+0.1} ${stand_depth/2-0.1} ${-stand_height*0.05}" rpy="0 0 0" />
-  </joint>
-  <link name="stand_leg_2">
-    <visual>
-      <origin xyz="0 0 0" rpy="0 0 0" />
-      <geometry>
-        <cylinder radius="0.05" length="${stand_height*0.1}" />
-      </geometry>
-      <material name="DarkGray" />
-    </visual>
-  </link>
-  <joint name="stand_to_leg_2" type="fixed">
-    <parent link="stand_base" />
-    <child link="stand_leg_2" />
-    <origin xyz="${stand_width/2-0.1} ${stand_depth/2-0.1} ${-stand_height*0.05}" rpy="0 0 0" />
-  </joint>
-  <link name="stand_leg_3">
-    <visual>
-      <origin xyz="0 0 0" rpy="0 0 0" />
-      <geometry>
-        <cylinder radius="0.05" length="${stand_height*0.1}" />
-      </geometry>
-      <material name="DarkGray" />
-    </visual>
-  </link>
-  <joint name="stand_to_leg_3" type="fixed">
-    <parent link="stand_base" />
-    <child link="stand_leg_3" />
-    <origin xyz="${-stand_width/2+0.1} ${-stand_depth/2+0.1} ${-stand_height*0.05}" rpy="0 0 0" />
-  </joint>
-  <link name="stand_leg_4">
-    <visual>
-      <origin xyz="0 0 0" rpy="0 0 0" />
-      <geometry>
-        <cylinder radius="0.05" length="${stand_height*0.1}" />
-      </geometry>
-      <material name="DarkGray" />
-    </visual>
-  </link>
-  <joint name="stand_to_leg_4" type="fixed">
-    <parent link="stand_base" />
-    <child link="stand_leg_4" />
-    <origin xyz="${stand_width/2-0.1} ${-stand_depth/2+0.1} ${-stand_height*0.05}" rpy="0 0 0" />
-  </joint>
-  <!-- Connect stand to world -->
-  <joint name="ground_to_stand" type="fixed">
-    <parent link="ground_plane" />
-    <child link="stand_base" />
-    <origin xyz="0 0 0" rpy="0 0 0" />
-  </joint>
-  <!-- Linear rail link -->
-  <link name="linear_rail">
-    <visual>
-      <origin xyz="0 0 0" rpy="0 0 0" />
-      <geometry>
-        <box size="${rail_length} ${rail_width} ${rail_height}" />
-      </geometry>
-      <material name="Black">
-        <color rgba="0.1 0.1 0.1 1.0" />
-      </material>
-    </visual>
-    <collision>
-      <origin xyz="0 0 0" rpy="0 0 0" />
-      <geometry>
-        <box size="${rail_length} ${rail_width} ${rail_height}" />
-      </geometry>
-    </collision>
-    <inertial>
-      <mass value="5.0" />
-      <inertia ixx="0.1" ixy="0.0" ixz="0.0" iyy="0.1" iyz="0.0" izz="0.1" />
-    </inertial>
-  </link>
-  <!-- Connect rail to stand -->
-  <joint name="stand_to_rail" type="fixed">
-    <parent link="stand_base" />
+        <color rgba="0.34 0.34 0.34 1.0" />
+      </material>
+    </visual>
+    <collision>
+      <origin xyz="0 0 0" rpy="0 0 0" />
+      <geometry>
+        <mesh filename="file://$(find ur_rail_description)/meshes/workspace/linear_rail.stl" scale="0.001 0.001 0.001"/>
+      </geometry>
+    </collision>
+    <inertial>
+      <mass value="10.0" />
+      <inertia ixx="1.0" ixy="0.0" ixz="0.0" iyy="1.0" iyz="0.0" izz="1.0" />
+    </inertial>
+  </link>
+  <!-- Connect linear rail to world -->
+  <joint name="ground_to_rail" type="fixed">
+    <parent link="work_cell" />
     <child link="linear_rail" />
-    <origin xyz="0 0 ${stand_height + rail_height/2}" rpy="0 0 0" />
+    <origin xyz="0 -0.48 0.79" rpy="0 0 0" />
   </joint>
   <!-- Slider base for robot -->
@@ -250,14 +269,14 @@
       <origin xyz="0 0 0" rpy="0 0 0" />
       <geometry>
-        <box size="0.2 0.2 0.05" />
-      </geometry>
-      <material name="Blue">
-        <color rgba="0.0 0.0 0.8 1.0" />
-      </material>
-    </visual>
-    <collision>
-      <origin xyz="0 0 0" rpy="0 0 0" />
-      <geometry>
-        <box size="0.2 0.2 0.05" />
+        <mesh filename="file://$(find ur_rail_description)/meshes/workspace/slider_base.stl" scale="0.001 0.001 0.001"/>
+      </geometry>
+      <material name="tin_alloy">
+        <color rgba="0.5 0.45 0.3 1.0" />
+      </material>
+    </visual>
+    <collision>
+      <origin xyz="0 0 0" rpy="0 0 0" />
+      <geometry>
+        <mesh filename="file://$(find ur_rail_description)/meshes/workspace/slider_base.stl" scale="0.001 0.001 0.001"/>
       </geometry>
     </collision>
@@ -271,7 +290,7 @@
     <parent link="linear_rail" />
     <child link="slider_base" />
-    <origin xyz="${0.1-rail_length/2} 0 ${rail_height/2}" rpy="0 0 0" />
+    <origin xyz="0 0 ${(slider_height+rail_height)/2}" rpy="0 0 0" />
     <axis xyz="1 0 0" />
-    <limit lower="0" upper="${rail_length-0.2}" effort="1000" velocity="0.5" />
+    <limit lower="-0.686" upper="0.686" effort="1000" velocity="0.5" />
     <dynamics damping="50.0" friction="1.0" />
   </joint> -->
@@ -279,5 +298,5 @@
     <parent link="linear_rail" />
     <child link="slider_base" />
-    <origin xyz="${0.1-rail_length/2} 0 ${rail_height/2}" rpy="0 0 0" />
+    <origin xyz="0 0 0.086" rpy="0 0 0" />
   </joint>
   <xacro:if value="$(arg sim_gazebo)">
@@ -296,6 +315,5 @@
     </gazebo>
     <gazebo>
-      <plugin filename="libign_ros2_control-system.so"
-        name="ign_ros2_control::IgnitionROS2ControlPlugin">
+      <plugin filename="gz_ros2_control-system" name="gz_ros2_control::GazeboSimROS2ControlPlugin">
         <parameters>$(arg simulation_controllers)</parameters>
         <controller_manager_node_name>$(arg tf_prefix)controller_manager</controller_manager_node_name>
