Commit message: Refactor RViz configuration and add camera macros
- Updated RViz configuration to improve panel layout and visibility settings.
- Added a new Xacro file for camera macros, defining standard camera and depth camera configurations.
- Introduced a materials Xacro file to define common materials used in URDF models.
- Modified the URDF for the UR on rail to include camera macros and materials, enhancing the robot's visual representation.
- Cleaned up mesh references and improved formatting for better readability.

File: urdf/ur_on_rail.urdf.xacro (robot description, xacro)
@@ -3,4 +3,6 @@
   <!-- Import the standard UR5 macro -->
   <xacro:include filename="$(find ur_rail_description)/urdf/ur_macro.xacro" />
+  <xacro:include filename="$(find ur_rail_description)/urdf/materials.xacro" />
+  <xacro:include filename="$(find ur_rail_description)/urdf/camera_macro.xacro" />
   <!-- Define properties for the linear rail and stand -->
   <xacro:property name="rail_length" value="1.5" />  <!-- Length of the rail -->
@@ -13,6 +15,4 @@
   <xacro:property name="slider_height" value="0.05" />
   <xacro:arg name="name" default="ur" />
-  <!-- import main macro -->
-  <xacro:include filename="$(find ur_rail_description)/urdf/ur_macro.xacro" />
   <!-- possible 'ur_type' values: ur3, ur3e, ur5, ur5e, ur7e, ur10, ur10e, ur12e, ur16e, ur20, ur30 -->
   <!-- the default value should raise an error in case this was called without defining the type -->
@@ -72,5 +72,6 @@
       <origin rpy="0 0 1.5707" xyz="0 0 -0.1" />
       <geometry>
-        <mesh filename="file://$(find ur_rail_description)/meshes/workspace/work_cell.stl" scale="0.001 0.001 0.001"/>
+        <mesh filename="file://$(find ur_rail_description)/meshes/workspace/work_cell.stl"
+          scale="0.001 0.001 0.001" />
       </geometry>
       <material name="ground_black">
@@ -81,5 +82,6 @@
       <origin rpy="0 0 1.5707" xyz="0 0 -0.1" />
       <geometry>
-        <mesh filename="file://$(find ur_rail_description)/meshes/workspace/work_cell.stl" scale="0.001 0.001 0.001"/>
+        <mesh filename="file://$(find ur_rail_description)/meshes/workspace/work_cell.stl"
+          scale="0.001 0.001 0.001" />
       </geometry>
     </collision>
@@ -130,9 +132,11 @@
     <origin xyz="0 0 0" rpy="0 0 0" />
   </xacro:ur_robot>
-  <link name="hex_qc_ft_sensor">
+  <!-- <link name="hex_qc_ft_sensor">
     <visual>
       <origin xyz="-0.058 -0.02 -0.03" rpy="1.5707 0 3.1414" />
       <geometry>
-        <mesh filename="file://$(find ur_rail_description)/meshes/onrobot_hex_qc_rg2/visual/HEX_E_H_QC_v3.dae" scale="0.001 0.001 0.001"/>
+        <mesh filename="file://$(find
+  ur_rail_description)/meshes/onrobot_hex_qc_rg2/visual/HEX_E_H_QC_v3(1).dae" scale="0.001 0.001
+  0.001"/>
       </geometry>
       <material name="White">
@@ -143,5 +147,7 @@
       <origin xyz="-0.058 -0.02 -0.03" rpy="1.5707 0 3.1414" />
       <geometry>
-        <mesh filename="file://$(find ur_rail_description)/meshes/onrobot_hex_qc_rg2/collision/HEX_E_H_QC_v3.stl" scale="0.001 0.0015 0.001"/>
+        <mesh filename="file://$(find
+  ur_rail_description)/meshes/onrobot_hex_qc_rg2/collision/HEX_E_H_QC_v3(1).stl" scale="0.001 0.0015
+  0.001"/>
       </geometry>
     </collision>
@@ -155,19 +161,19 @@
     <child link="hex_qc_ft_sensor" />
     <origin xyz="0 0 0" rpy="0 0 0" />
-  </joint>
+  </joint> -->
   <link name="plc_linear_rail">
     <visual>
       <origin xyz="0 0 0.884" rpy="0 0 0" />
       <geometry>
-        <mesh filename="file://$(find ur_rail_description)/meshes/workspace/plc_linear_rail.stl" scale="0.001 0.001 0.001"/>
-      </geometry>
-      <material name="White">
-        <color rgba="0.79 0.79 0.79 1.0" />
-      </material>
+        <mesh filename="file://$(find ur_rail_description)/meshes/workspace/plc_linear_rail.stl"
+          scale="0.001 0.001 0.001" />
+      </geometry>
+      <material name="Aluminium" />
     </visual>
     <collision>
       <origin xyz="0 0 0.884" rpy="0 0 0" />
       <geometry>
-        <mesh filename="file://$(find ur_rail_description)/meshes/workspace/plc_linear_rail.stl" scale="0.001 0.001 0.001"/>
+        <mesh filename="file://$(find ur_rail_description)/meshes/workspace/plc_linear_rail.stl"
+          scale="0.001 0.001 0.001" />
       </geometry>
     </collision>
@@ -187,14 +193,14 @@
       <origin xyz="0 0 0" rpy="0 0 0" />
       <geometry>
-        <mesh filename="file://$(find ur_rail_description)/meshes/workspace/table.stl" scale="0.001 0.001 0.001"/>
-      </geometry>
-      <material name="Aluminium">
-        <color rgba="0.78 0.78 0.78 1.0" />
-      </material>
-    </visual>
-    <collision>
-      <origin xyz="0 0 0" rpy="0 0 0" />
-      <geometry>
-        <mesh filename="file://$(find ur_rail_description)/meshes/workspace/table.stl" scale="0.001 0.001 0.001"/>
+        <mesh filename="file://$(find ur_rail_description)/meshes/workspace/table.stl"
+          scale="0.001 0.001 0.001" />
+      </geometry>
+      <material name="Aluminium" />
+    </visual>
+    <collision>
+      <origin xyz="0 0 0" rpy="0 0 0" />
+      <geometry>
+        <mesh filename="file://$(find ur_rail_description)/meshes/workspace/table.stl"
+          scale="0.001 0.001 0.001" />
       </geometry>
     </collision>
@@ -208,14 +214,14 @@
       <origin xyz="0 0 0" rpy="0 0 0" />
       <geometry>
-        <mesh filename="file://$(find ur_rail_description)/meshes/workspace/table.stl" scale="0.001 0.001 0.001"/>
-      </geometry>
-      <material name="Aluminium">
-        <color rgba="0.78 0.78 0.78 1.0" />
-      </material>
-    </visual>
-    <collision>
-      <origin xyz="0 0 0" rpy="0 0 0" />
-      <geometry>
-        <mesh filename="file://$(find ur_rail_description)/meshes/workspace/table.stl" scale="0.001 0.001 0.001"/>
+        <mesh filename="file://$(find ur_rail_description)/meshes/workspace/table.stl"
+          scale="0.001 0.001 0.001" />
+      </geometry>
+      <material name="Aluminium" />
+    </visual>
+    <collision>
+      <origin xyz="0 0 0" rpy="0 0 0" />
+      <geometry>
+        <mesh filename="file://$(find ur_rail_description)/meshes/workspace/table.stl"
+          scale="0.001 0.001 0.001" />
       </geometry>
     </collision>
@@ -229,5 +235,5 @@
     <parent link="work_cell" />
     <child link="table1" />
-    <origin xyz="0.34 0.3 0.74" rpy="0 0 0" />
+    <origin xyz="0.86 0.25 0.74" rpy="0 0 0" />
   </joint>
   <!-- Connect table2 to world -->
@@ -235,5 +241,5 @@
     <parent link="work_cell" />
     <child link="table2" />
-    <origin xyz="-0.34 0.3 0.74" rpy="0 0 0" />
+    <origin xyz="0.0 0.17 0.74" rpy="0 0 0" />
   </joint>
   <link name="linear_rail">
@@ -241,5 +247,6 @@
       <origin xyz="0 0 0" rpy="0 0 0" />
       <geometry>
-        <mesh filename="file://$(find ur_rail_description)/meshes/workspace/linear_rail.stl" scale="0.001 0.001 0.001"/>
+        <mesh filename="file://$(find ur_rail_description)/meshes/workspace/linear_rail.stl"
+          scale="0.001 0.001 0.001" />
       </geometry>
       <material name="DarkGray">
@@ -250,5 +257,6 @@
       <origin xyz="0 0 0" rpy="0 0 0" />
       <geometry>
-        <mesh filename="file://$(find ur_rail_description)/meshes/workspace/linear_rail.stl" scale="0.001 0.001 0.001"/>
+        <mesh filename="file://$(find ur_rail_description)/meshes/workspace/linear_rail.stl"
+          scale="0.001 0.001 0.001" />
       </geometry>
     </collision>
@@ -269,5 +277,6 @@
       <origin xyz="0 0 0" rpy="0 0 0" />
       <geometry>
-        <mesh filename="file://$(find ur_rail_description)/meshes/workspace/slider_base.stl" scale="0.001 0.001 0.001"/>
+        <mesh filename="file://$(find ur_rail_description)/meshes/workspace/slider_base.stl"
+          scale="0.001 0.001 0.001" />
       </geometry>
       <material name="tin_alloy">
@@ -278,5 +287,6 @@
       <origin xyz="0 0 0" rpy="0 0 0" />
       <geometry>
-        <mesh filename="file://$(find ur_rail_description)/meshes/workspace/slider_base.stl" scale="0.001 0.001 0.001"/>
+        <mesh filename="file://$(find ur_rail_description)/meshes/workspace/slider_base.stl"
+          scale="0.001 0.001 0.001" />
       </geometry>
     </collision>
@@ -300,4 +310,18 @@
     <origin xyz="0 0 0.086" rpy="0 0 0" />
   </joint>
+  <!-- RGB Cameras -->
+  <xacro:camera_macro name="camera_1">
+    <origin xyz="1.0 -0.7 2.0" rpy="0 0.8 2.50" />
+  </xacro:camera_macro>
+  <xacro:camera_macro name="camera_2">
+    <origin xyz="-1.0 -0.7 2.0" rpy="0 0.8 0.64" />
+  </xacro:camera_macro>
+  <xacro:camera_macro name="camera_3">
+    <origin xyz="0 1.0 2.0" rpy="0 1.0 -1.5707" />
+  </xacro:camera_macro>
+  <!-- Depth Cameras -->
+  <xacro:depth_camera_macro name="depth_camera">
+    <origin xyz="0 0 3" rpy="0 1.5707 0" />
+  </xacro:depth_camera_macro>
   <xacro:if value="$(arg sim_gazebo)">
     <!-- Gazebo plugins -->
@@ -312,7 +336,11 @@
   <xacro:if value="$(arg sim_ignition)">
     <!-- Gazebo plugins -->
-    <gazebo reference="world">
-    </gazebo>
+    <gazebo reference="world"></gazebo>
     <gazebo>
+      <plugin
+        filename="ignition-gazebo-sensors-system"
+        name="gz::sim::systems::Sensors">
+        <render_engine>ogre2</render_engine>
+      </plugin>
       <plugin filename="gz_ros2_control-system" name="gz_ros2_control::GazeboSimROS2ControlPlugin">
         <parameters>$(arg simulation_controllers)</parameters>

Commit message: Repositioned Oak camera 1

File: urdf/ur_on_rail.urdf.xacro (robot description, xacro)
@@ -312,5 +312,5 @@
   <!-- RGB Cameras -->
   <xacro:camera_macro name="camera_1">
-    <origin xyz="1.0 -0.7 2.0" rpy="0 0.8 2.50" />
+    <origin xyz="0.86 0.25 1.0" rpy="0 0 3.1414" />
   </xacro:camera_macro>
   <xacro:camera_macro name="camera_2">
