Commit message: Add OAK-1 mesh and update camera macros with new properties

File: urdf/camera_macro.xacro (robot description, xacro)
@@ -4,7 +4,10 @@
         <link name="${name}">
             <visual>
+                <origin xyz="-0.02 -0.0176 -0.032" rpy="1.5707 0 1.5707" />
                 <geometry>
-                    <box size="0.05 0.05 0.05" />
+                    <mesh filename="file://$(find ur_rail_description)/meshes/oak_camera/OAK-1.stl"
+                        scale="0.001 0.001 0.001" />
                 </geometry>
+                <material name="Black" />
             </visual>
             <collision>
@@ -62,4 +65,5 @@
                     <box size="0.05 0.05 0.05" />
                 </geometry>
+                <material name="Black" />
             </visual>
             <collision>

File: urdf/materials.xacro (robot description, xacro)
@@ -4,3 +4,6 @@
         <color rgba="0.6 0.6 0.6 1.0" />
     </material>
+    <material name="Black">
+        <color rgba="0.7 0.7 0.7 1" />
+    </material>
 </robot>

File: urdf/ur_on_rail.urdf.xacro (robot description, xacro)
@@ -318,5 +318,5 @@
   </xacro:camera_macro>
   <xacro:camera_macro name="camera_3">
-    <origin xyz="0 1.0 2.0" rpy="0 1.0 -1.5707" />
+    <origin xyz="0 1.0 2.0" rpy="0 0 -1.5707" />
   </xacro:camera_macro>
   <!-- Depth Cameras -->

Commit message: Update camera configurations and rename camera macros for clarity

File: urdf/camera_macro.xacro (robot description, xacro)
@@ -26,8 +26,8 @@
             <xacro:insert_block name="origin" />
         </joint>
-        <link name="${name}_optical" />
+        <link name="${name}_optical_frame" />
         <joint name="${name}_optical_joint" type="fixed">
             <parent link="${name}" />
-            <child link="${name}_optical" />
+            <child link="${name}_optical_frame" />
             <origin xyz="0 0 0" rpy="-1.5707 0 -1.5707" />
         </joint>

File: urdf/ur_on_rail.urdf.xacro (robot description, xacro)
@@ -311,11 +311,11 @@
   </joint>
   <!-- RGB Cameras -->
-  <xacro:camera_macro name="camera_1">
-    <origin xyz="0.86 0.25 1.0" rpy="0 0 3.1414" />
+  <xacro:camera_macro name="oak1_rgb_camera">
+    <origin xyz="0.862 0.17 1.175" rpy="-0.005 0.455 3.095" />
   </xacro:camera_macro>
-  <xacro:camera_macro name="camera_2">
+  <xacro:camera_macro name="oak2_rgb_camera">
     <origin xyz="-1.0 -0.7 2.0" rpy="0 0.8 0.64" />
   </xacro:camera_macro>
-  <xacro:camera_macro name="camera_3">
+  <xacro:camera_macro name="oak3_rgb_camera">
     <origin xyz="0 1.0 2.0" rpy="0 0 -1.5707" />
   </xacro:camera_macro>
